File: pcbs/keyboard.kicad_pcb (KiCad board)
At the start: 2 copper layers, 160 parts, among them J1 MJ-4PP-9, J2 MJ-4PP-9, SW1 SW_PUSH, SW2 SW_PUSH, U1 Arduino_Pro_Micro, U2 Arduino_Pro_Micro

Commit message: Updated pcbs.
Parts:
- added G***: LOGO, LOGO, F.Cu at (82.5, 184.9)
- added Ref**: Val**, kbd:M2_HOLE_v2, F.Cu at (392.9, 112.7)
- added Ref**: Val**, kbd:M2_HOLE_v2, F.Cu at (388.1, 200.8)
- added Ref**: Val**, kbd:M2_HOLE_v2, F.Cu at (297.6, 162.7)
- added Ref**: Val**, kbd:M2_HOLE_v2, F.Cu at (191.3, 112.7)
- added Ref**: Val**, kbd:M2_HOLE_v2, F.Cu at (215.1, 200.8)
- added Ref**: Val**, kbd:M2_HOLE_v2, F.Cu at (340.5, 200.8)
- added Ref**: Val**, kbd:M2_HOLE_v2, F.Cu at (373.0, 162.7)
- added Ref**: Val**, kbd:M2_HOLE_v2, F.Cu at (153.2, 112.7)
- added Ref**: Val**, kbd:M2_HOLE_v2, F.Cu at (130.2, 162.7)
- added Ref**: Val**, kbd:M2_HOLE_v2, F.Cu at (119.8, 200.8)
- added Ref**: Val**, kbd:M2_HOLE_v2, F.Cu at (167.5, 200.8)
- added Ref**: Val**, kbd:M2_HOLE_v2, F.Cu at (115.1, 143.7)
- added Ref**: Val**, kbd:M2_HOLE_v2, F.Cu at (352.4, 112.7)
- added Ref**: Val**, kbd:M2_HOLE_v2, F.Cu at (388.9, 143.7)
- added Ref**: Val**, kbd:M2_HOLE_v2, F.Cu at (274.6, 112.7)
- added Ref**: Val**, kbd:M2_HOLE_v2, F.Cu at (162.7, 143.7)
- added Ref**: Val**, kbd:M2_HOLE_v2, F.Cu at (278.6, 143.7)
- added Ref**: Val**, kbd:M2_HOLE_v2, F.Cu at (210.3, 143.7)
- added Ref**: Val**, kbd:M2_HOLE_v2, F.Cu at (229.4, 269.9)
- added Ref**: Val**, kbd:M2_HOLE_v2, F.Cu at (335.7, 143.7)
- added Ref**: Val**, kbd:M2_HOLE_v2, F.Cu at (283.4, 200.8)
- added Ref**: Val**, kbd:M2_HOLE_v2, F.Cu at (115.1, 112.7)
- added Ref**: Val**, kbd:M2_HOLE_v2, F.Cu at (200.8, 162.7)
- U1: moved to F.Cu
- moved U1 32.6 mm to (220.2, 111.4), turned to 0 degrees
- moved J1 32.6 mm to (233.3, 93.6)
- moved SW1 32.6 mm to (233.3, 111.9)
- moved D_19 32.6 mm to (161.1, 173.0)
- moved D_20 32.6 mm to (180.2, 173.0)
- moved D_21 32.6 mm to (199.2, 173.0)
- moved D_22 32.6 mm to (218.3, 173.0)
- moved D_34 32.6 mm to (218.3, 211.1)
- moved K_1 32.6 mm to (162.7, 103.1)
- moved K_16 32.6 mm to (210.3, 153.2)
- moved K_20 32.6 mm to (177.0, 172.2)
- moved K_27 32.6 mm to (186.5, 191.3)
- moved K_29 32.6 mm to (224.6, 191.3)
- moved K_3 32.6 mm to (200.8, 103.1)
- moved K_7 32.6 mm to (162.7, 134.1)
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Routing:
- net row5_r: track 283.2 -> 0.00 mm
- net row4_r: track 270.6 -> 0.00 mm
- net row3_r: track 238.8 -> 0.00 mm
- net row2_r: track 238.4 -> 0.00 mm
- net col0: track 224.4 -> 0.00 mm, vias 1 -> 0
- net row6: track 213.2 -> 0.00 mm
- net row5: track 196.9 -> 0.00 mm
- net col7_r: track 192.9 -> 0.00 mm, vias 1 -> 0
- net col1: track 188.0 -> 0.00 mm
- net col2: track 168.9 -> 0.00 mm
- net col6_r: track 165.1 -> 0.00 mm, vias 1 -> 0
- net row4: track 163.7 -> 0.00 mm
- net col1_r: track 156.1 -> 0.00 mm, vias 1 -> 0
- net row0_r: track 155.8 -> 0.00 mm
- net col0_r: track 154.8 -> 0.00 mm, vias 1 -> 0
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Other:
- board text added: "Fatotesa Keyboard rev.1"

Commit message: Use smd+through hole diode footprint.
Parts:
- removed G***: LOGO, LOGO
- removed Ref** (x23): Val**, kbd:M2_HOLE_v2
- removed U2: Arduino_Pro_Micro, ScottoKeebs_MCU:Arduino_Pro_Micro
- added U3: ProMicro, Corne:ProMicro_v3, F.Cu at (220.3, 109.5)
- D_0, D_1, D_10, D_11, D_12, D_13, D_14, D_15, D_16, D_17, D_18, D_19, D_2, D_20, D_21, D_22, D_23, D_24, D_25, D_26, D_27, D_28, D_29, D_3, D_30, D_31, D_32, D_33, D_34, D_35, D_36, D_37, D_38, D_39, D_4, D_40, D_41, D_42, D_43, D_44, D_45, D_46, D_47, D_48, D_49, D_5, D_50, D_51, D_52, D_53, D_54, D_55, D_56, D_57, D_58, D_59, D_6, D_60, D_61, D_62, D_63, D_64, D_65, D_66, D_67, D_68, D_69, D_7, D_70, D_71, D_72, D_73, D_74, D_8, D_9: footprint Diode_SMD:D_SOD-123 -> Corne:D3_TH_SMD_v2
- U1: value Arduino_Pro_Micro -> ProMicro; footprint ScottoKeebs_MCU:Arduino_Pro_Micro -> Corne:ProMicro_v3
- moved U1 134.5 mm to (354.6, 109.6)
- moved J2 32.1 mm to (283.1, 91.2)
- moved D_63 31.8 mm to (396.9, 104.0)
- moved D_35 31.8 mm to (299.9, 104.0)
- moved D_37 31.8 mm to (318.9, 104.0)
- moved D_42 31.8 mm to (338.0, 104.0)
- moved D_57 31.8 mm to (377.8, 104.0)
- moved D_68 31.8 mm to (415.9, 104.0)
- moved K_35 31.7 mm to (296.7, 103.2)
- moved K_41 31.7 mm to (305.6, 191.3)
- moved K_42 31.7 mm to (334.8, 103.2)
- moved K_51 31.7 mm to (343.7, 191.3)
- moved K_61 31.7 mm to (381.8, 191.3)
- moved K_62 31.7 mm to (384.2, 210.3)
- moved K_74 31.7 mm to (431.8, 210.3)
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Connections:
- U1 pad 10: row4 -> row3_r
- U1 pad 11: row3 -> row2_r
- U1 pad 12: row2 -> row1_r
- U1 pad 13: col6 -> col3_r
- U1 pad 14: col5 -> row4_r
- U1 pad 15: col4 -> row5_r
- U1 pad 16: col3 -> col4_r
- U1 pad 17: col2 -> col5_r
- U1 pad 18: col1 -> col6_r
- U1 pad 19: col0 -> col7_r
- U1 pad 2: data -> data_r
- U1 pad 20: row0 -> row0_r
- U1 pad 21: VCC -> VDD
- U1 pad 22: reset -> reset_r
- U1 pad 23: GND -> GNDA
- U1 pad 3: GND -> GNDA
- U1 pad 4: GND -> GNDA
- U1 pad 7: unconnected-(U1-4/PD4-Pad7) -> col2_r
- U1 pad 8: row6 -> col1_r
- U1 pad 9: row5 -> col0_r
Other:
- board outline added: 188.3 x 134.1 mm
- board text removed: "Fatotesa Keyboard rev.1"

Commit message: Fixed board outlines + breakout pads.
Parts:
- added ?: , , F.Cu at (210.3, 225.4)
- added ?: , , F.Cu at (142.1, 90.5)
- added ?: , , F.Cu at (415.1, 90.5)
- added ?: , , F.Cu at (414.3, 90.5)
- added ?: , , F.Cu at (305.6, 90.5)
- added ?: , , F.Cu at (102.4, 225.4)
- added ?: , , F.Cu at (140.5, 90.5)
- added ?: , , F.Cu at (310.3, 225.4)
- added ?: , , F.Cu at (88.9, 90.5)
- added ?: , , F.Cu at (308.0, 90.5)
- added ?: , , F.Cu at (347.6, 90.5)
- added ?: , , F.Cu at (308.7, 225.4)
- added ?: , , F.Cu at (309.5, 225.4)
- added ?: , , F.Cu at (426.2, 225.4)
- added ?: , , F.Cu at (89.7, 90.5)
- added ?: , , F.Cu at (205.6, 90.5)
- added ?: , , F.Cu at (207.2, 90.5)
- added ?: , , F.Cu at (208.7, 90.5)
- added ?: , , F.Cu at (311.9, 90.5)
- added ?: , , F.Cu at (208.7, 225.4)
- added ?: , , F.Cu at (177.0, 225.4)
- added ?: , , F.Cu at (310.3, 90.5)
- added ?: , , F.Cu at (100.8, 225.4)
- added ?: , , F.Cu at (138.9, 90.5)
- added ?: , , F.Cu at (103.2, 225.4)
- added ?: , , F.Cu at (429.4, 225.4)
- added ?: , , F.Cu at (311.1, 90.5)
- added ?: , , F.Cu at (377.0, 225.4)
- added ?: , , F.Cu at (307.2, 225.4)
- added ?: , , F.Cu at (170.6, 225.4)
- added ?: , , F.Cu at (92.1, 90.5)
- added ?: , , F.Cu at (419.1, 90.5)
- added ?: , , F.Cu at (213.5, 225.4)
- added ?: , , F.Cu at (209.5, 90.5)
- added ?: , , F.Cu at (100.0, 225.4)
- added ?: , , F.Cu at (308.7, 90.5)
- added ?: , , F.Cu at (87.3, 90.5)
- added ?: , , F.Cu at (143.7, 90.5)
- added ?: , , F.Cu at (141.3, 90.5)
- added ?: , , F.Cu at (210.3, 90.5)
- added ?: , , F.Cu at (307.2, 90.5)
- added ?: , , F.Cu at (381.8, 225.4)
- added ?: , , F.Cu at (173.0, 225.4)
- added ?: , , F.Cu at (88.1, 90.5)
- added ?: , , F.Cu at (175.4, 225.4)
- added ?: , , F.Cu at (348.4, 90.5)
- added ?: , , F.Cu at (342.9, 90.5)
- added ?: , , F.Cu at (207.2, 225.4)
- added ?: , , F.Cu at (431.0, 225.4)
- added ?: , , F.Cu at (308.0, 225.4)
- added ?: , , F.Cu at (106.4, 225.4)
- added ?: , , F.Cu at (417.5, 90.5)
- added ?: , , F.Cu at (206.4, 90.5)
- added ?: , , F.Cu at (381.0, 225.4)
- added ?: , , F.Cu at (171.4, 225.4)
- added ?: , , F.Cu at (90.5, 90.5)
- added ?: , , F.Cu at (207.9, 90.5)
- added ?: , , F.Cu at (376.2, 225.4)
- added ?: , , F.Cu at (309.5, 90.5)
- added ?: , , F.Cu at (427.8, 225.4)
- added ?: , , F.Cu at (312.7, 225.4)
- added ?: , , F.Cu at (174.6, 225.4)
- added ?: , , F.Cu at (412.7, 90.5)
- added ?: , , F.Cu at (142.9, 90.5)
- added ?: , , F.Cu at (311.1, 225.4)
- added ?: , , F.Cu at (104.0, 225.4)
- added ?: , , F.Cu at (416.7, 90.5)
- added ?: , , F.Cu at (138.1, 90.5)
- added ?: , , F.Cu at (176.2, 225.4)
- added ?: , , F.Cu at (207.9, 225.4)
- added ?: , , F.Cu at (428.6, 225.4)
- added ?: , , F.Cu at (137.3, 90.5)
- added ?: , , F.Cu at (306.4, 90.5)
- added ?: , , F.Cu at (427.0, 225.4)
- added ?: , , F.Cu at (375.4, 225.4)
- added ?: , , F.Cu at (425.4, 225.4)
- added ?: , , F.Cu at (211.9, 90.5)
- added ?: , , F.Cu at (345.3, 90.5)
- added ?: , , F.Cu at (212.7, 225.4)
- added ?: , , F.Cu at (418.3, 90.5)
- added ?: , , F.Cu at (104.8, 225.4)
- added ?: , , F.Cu at (344.5, 90.5)
- added ?: , , F.Cu at (415.9, 90.5)
- added ?: , , F.Cu at (91.3, 90.5)
- added ?: , , F.Cu at (431.8, 225.4)
- added ?: , , F.Cu at (172.2, 225.4)
- added ?: , , F.Cu at (211.9, 225.4)
- added ?: , , F.Cu at (346.1, 90.5)
- added ?: , , F.Cu at (430.2, 225.4)
- added ?: , , F.Cu at (378.6, 225.4)
- added ?: , , F.Cu at (139.7, 90.5)
- added ?: , , F.Cu at (173.8, 225.4)
- added ?: , , F.Cu at (380.2, 225.4)
- added ?: , , F.Cu at (379.4, 225.4)
- added ?: , , F.Cu at (377.8, 225.4)
- added ?: , , F.Cu at (413.5, 90.5)
- added ?: , , F.Cu at (342.1, 90.5)
- added ?: , , F.Cu at (105.6, 225.4)
- added ?: , , F.Cu at (313.5, 225.4)
- added ?: , , F.Cu at (346.8, 90.5)
- added ?: , , F.Cu at (211.1, 90.5)
- added ?: , , F.Cu at (343.7, 90.5)
- added ?: , , F.Cu at (209.5, 225.4)
- added ?: , , F.Cu at (101.6, 225.4)
- added ?: , , F.Cu at (311.9, 225.4)
- added ?: , , F.Cu at (93.7, 90.5)
- added ?: , , F.Cu at (211.1, 225.4)
- added ?: , , F.Cu at (92.9, 90.5)
- added SW3: RotaryEncoder_Switch, Keebio-Parts:RotaryEncoder_Alps_EC11E-Switch_Vertical_H20mm, F.Cu at (83.3, 103.2)
Routing:
- net col7_r: track 0.00 -> 120.5 mm
- net col4: track 0.00 -> 119.0 mm
- net row5: track 0.00 -> 116.7 mm
- net col1_r: track 0.00 -> 115.8 mm
- net row2: track 0.00 -> 115.2 mm
- net col4_r: track 0.00 -> 115.0 mm
- net col6_r: track 0.00 -> 115.0 mm
- net col0: track 0.00 -> 112.1 mm
- net row6: track 0.00 -> 108.0 mm
- net row4: track 0.00 -> 102.4 mm
- net row3: track 0.00 -> 100.0 mm
- net col3: track 0.00 -> 98.0 mm
- net col5: track 0.00 -> 98.0 mm
- net row0: track 0.00 -> 97.2 mm
- net col2_r: track 0.00 -> 95.7 mm
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Other:
- board size 188.3 x 134.1 mm -> 404.9 x 152.4 mm
- board text added: "2023/24"
- board text added: "FATO-TESA-KBD rev.1"

Commit message: Added CU fill and other stuff.
Parts:
- removed ? (x108): , 
- added D_75: D, Corne:D3_TH_SMD_v2, B.Cu at (146.8, 103.8)
- added G***: LOGO, LOGO, F.Cu at (84.9, 156.4)
- added G***: LOGO, LOGO, B.Cu at (84.9, 156.4)
- S2, S3: footprint PCM_marbastlib-mx:STAB_MX_P_2.75u -> PCM_marbastlib-mx:STAB_MX_P_2u
- moved SW3 52.4 mm to (135.7, 103.2)
Connections:
- SW3 pad A: unconnected-(SW3-PadA) -> encA
- SW3 pad B: unconnected-(SW3-PadB) -> encB
- SW3 pad C: unconnected-(SW3-PadC) -> GND
- SW3 pad S1: unconnected-(SW3-PadS1) -> col1
- SW3 pad S2: unconnected-(SW3-PadS2) -> rotB
- U1 pad 10: row3_r -> col5_r
- U1 pad 11: row2_r -> col4_r
- U1 pad 12: row1_r -> col3_r
- U1 pad 13: col3_r -> row1_r
- U1 pad 14: row4_r -> row2_r
- U1 pad 15: row5_r -> row3_r
- U1 pad 16: col4_r -> row4_r
- U1 pad 17: col5_r -> row5_r
- U1 pad 18: col6_r -> col0_r
- U1 pad 19: col7_r -> col1_r
- U1 pad 20: row0_r -> col2_r
- U1 pad 7: col2_r -> row0_r
- U1 pad 8: col1_r -> col7_r
- U1 pad 9: col0_r -> col6_r
- U3 pad 10: unconnected-(U3-7/E6-Pad10) -> row4
- U3 pad 11: unconnected-(U3-8/B4-Pad11) -> row3
- U3 pad 12: unconnected-(U3-9/B5-Pad12) -> row2
- U3 pad 14: unconnected-(U3-B2/16-Pad14) -> col1
- U3 pad 15: unconnected-(U3-B3/14-Pad15) -> col2
- U3 pad 16: unconnected-(U3-B1/15-Pad16) -> col3
- U3 pad 17: unconnected-(U3-F7/A0-Pad17) -> col4
- U3 pad 18: unconnected-(U3-F6/A1-Pad18) -> col5
- U3 pad 19: unconnected-(U3-F5/A2-Pad19) -> col6
- U3 pad 8: unconnected-(U3-5/C6-Pad8) -> row6
- U3 pad 9: unconnected-(U3-6/D7-Pad9) -> row5
Routing:
- net row5_r: track 0.00 -> 296.4 mm
- net row4_r: track 0.00 -> 261.8 mm
- net row3_r: track 0.00 -> 242.9 mm
- net row2_r: track 0.00 -> 238.5 mm
- net row1_r: track 0.00 -> 175.4 mm
- net row0_r: track 0.00 -> 140.3 mm, vias 0 -> 1
- net col1: track 87.0 -> 202.0 mm, vias 0 -> 1
- net col0: track 112.1 -> 223.7 mm, vias 0 -> 1
- net row6: track 108.0 -> 216.9 mm
- net GND: track 0.00 -> 105.4 mm
- net col2: track 89.0 -> 174.1 mm, vias 0 -> 1
- net VDD: track 0.00 -> 82.4 mm, vias 0 -> 1
- net row5: track 116.7 -> 198.9 mm
- net GNDA: track 0.00 -> 80.6 mm
- net data_r: track 0.00 -> 78.7 mm
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- added copper zone on B.Cu, net (none)
- added copper zone on F.Cu, net (none)
Other:
- board text added: "www.fatotesa.se - split keyboard - rev 2023.1"

Commit message: Added LEDs for underglow.
Parts:
- added LED1: WS2812B, LED_SMD:LED_WS2812B_PLCC4_5.0x5.0mm_P3.2mm, B.Cu at (96.9, 144.5)
- added LED10: WS2812B, LED_SMD:LED_WS2812B_PLCC4_5.0x5.0mm_P3.2mm, B.Cu at (415.9, 181.0)
- added LED11: WS2812B, LED_SMD:LED_WS2812B_PLCC4_5.0x5.0mm_P3.2mm, B.Cu at (367.6, 142.9)
- added LED12: WS2812B, LED_SMD:LED_WS2812B_PLCC4_5.0x5.0mm_P3.2mm, B.Cu at (420.6, 142.9)
- added LED2: WS2812B, LED_SMD:LED_WS2812B_PLCC4_5.0x5.0mm_P3.2mm, B.Cu at (98.4, 181.8)
- added LED3: WS2812B, LED_SMD:LED_WS2812B_PLCC4_5.0x5.0mm_P3.2mm, B.Cu at (153.2, 142.9)
- added LED4: WS2812B, LED_SMD:LED_WS2812B_PLCC4_5.0x5.0mm_P3.2mm, B.Cu at (157.9, 183.4)
- added LED5: WS2812B, LED_SMD:LED_WS2812B_PLCC4_5.0x5.0mm_P3.2mm, B.Cu at (211.1, 142.1)
- added LED6: WS2812B, LED_SMD:LED_WS2812B_PLCC4_5.0x5.0mm_P3.2mm, B.Cu at (215.1, 183.3)
- added LED7: WS2812B, LED_SMD:LED_WS2812B_PLCC4_5.0x5.0mm_P3.2mm, B.Cu at (315.1, 182.6)
- added LED8: WS2812B, LED_SMD:LED_WS2812B_PLCC4_5.0x5.0mm_P3.2mm, B.Cu at (366.6, 181.0)
- added LED9: WS2812B, LED_SMD:LED_WS2812B_PLCC4_5.0x5.0mm_P3.2mm, B.Cu at (311.9, 143.7)
Connections:
- U1 pad 1: unconnected-(U1-TX0/D3-Pad1) -> LED_r
- U3 pad 1: unconnected-(U3-TX0/D3-Pad1) -> LED
Routing:
- net GND: track 105.4 -> 475.6 mm, vias 0 -> 2
- net VCC: track 23.8 -> 375.5 mm, vias 1 -> 4
- net GNDA: track 80.6 -> 419.7 mm, vias 0 -> 4
- net VDD: track 82.4 -> 403.1 mm, vias 1 -> 2
- net Net-(LED3-DIN): track 0.00 -> 63.8 mm
- net Net-(LED1-DIN): track 0.00 -> 62.5 mm
- net Net-(LED11-DOUT): track 0.00 -> 61.8 mm
- net LED: track 0.00 -> 59.5 mm, vias 0 -> 1
- net Net-(LED2-DOUT): track 0.00 -> 55.2 mm
- net Net-(LED4-DOUT): track 0.00 -> 53.7 mm
- net Net-(LED7-DOUT): track 0.00 -> 52.8 mm
- net Net-(LED10-DOUT): track 0.00 -> 47.5 mm, vias 0 -> 2
- net LED_r: track 0.00 -> 47.4 mm, vias 0 -> 1
- net Net-(LED10-DIN): track 0.00 -> 45.8 mm
- net Net-(LED7-DIN): track 0.00 -> 40.7 mm, vias 0 -> 2
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