File: pcbs/keyboard.kicad_pcb (KiCad board)
At the start: 2 copper layers, 378.3 x 160.2 mm, 218 parts, among them J1 MJ-4PP-9, J2 MJ-4PP-9, SW1 SW_PUSH, SW2 SW_PUSH, SW3 RotaryEncoder_Switch, U1 ProMicro, U3 ProMicro

Commit message: Branch for a split jlcpcb order.
Parts:
- removed D_0, D_1, D_10, D_11, D_12, D_13, D_14, D_15, D_16, D_17, D_18, D_19, D_2, D_20, D_21, D_22, D_23, D_24, D_25, D_26, D_27, D_28, D_29, D_3, D_30, D_31, D_32, D_33, D_34, D_4, D_5, D_6, D_7, D_75, D_8, D_9: D, kbd:D3_TH
- removed the G*** at (197.6, 138.9)
- removed the G*** at (198.4, 138.9)
- removed H1, H10, H11, H12, H2, H3, H4, H5, H6, H7, H8, H9: MountingHole, MountingHole:MountingHole_4.3mm_M4
- removed H25, H26, H27, H31: MountingHole, MountingHole:MountingHole_5.3mm_M5
- removed H33, H34, H35, H36, H37, H38, H39, H40: MountingHole, Keebio-Parts:breakaway-mousebites_fat-o-tesa
- removed J1: MJ-4PP-9, Corne:MJ-4PP-9_1side
- removed K_0, K_1, K_10, K_12, K_13, K_14, K_15, K_16, K_18, K_19, K_2, K_20, K_21, K_22, K_24, K_25, K_26, K_27, K_28, K_29, K_3, K_34, K_4, K_5, K_6, K_7, K_8, K_9: KEYSW, MX_Only:MXOnly-1U-NoLED
- removed K_11: KEYSW, MX_Only:MXOnly-1.5U-NoLED
- removed K_17, K_33: KEYSW, MX_Only:MXOnly-1.75U-NoLED
- removed K_23, K_30, K_31, K_32: KEYSW, MX_Only:MXOnly-1.25U-NoLED
- removed LED1, LED2, LED3, LED4, LED5, LED6: WS2812B, LED_SMD:LED_WS2812B_PLCC4_5.0x5.0mm_P3.2mm
- removed SW1: SW_PUSH, kbd:ResetSMD_SG
- removed SW3: RotaryEncoder_Switch, Keebio-Parts:RotaryEncoder_Alps_EC11E-Switch_Vertical_H20mm
- removed U3: ProMicro, Corne:ProMicro_v3_inverted
Routing:
- net GND: track 583.9 -> 0.00 mm, vias 10 -> 0
- net VCC: track 433.0 -> 0.00 mm, vias 7 -> 0
- net reset: track 261.6 -> 0.00 mm
- net col6: track 236.5 -> 0.00 mm, vias 2 -> 0
- net row6: track 236.5 -> 0.00 mm, vias 1 -> 0
- net row5: track 232.7 -> 0.00 mm, vias 1 -> 0
- net col4: track 211.7 -> 0.00 mm, vias 1 -> 0
- net col5: track 208.8 -> 0.00 mm, vias 1 -> 0
- net row4: track 205.3 -> 0.00 mm, vias 1 -> 0
- net LED: track 201.9 -> 0.00 mm, vias 2 -> 0
- net row3: track 180.3 -> 0.00 mm, vias 2 -> 0
- net col3: track 171.1 -> 0.00 mm, vias 1 -> 0
- net row2: track 170.8 -> 0.00 mm, vias 2 -> 0
- net col1: track 167.7 -> 0.00 mm, vias 1 -> 0
- net data: track 161.7 -> 0.00 mm
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- added copper zone on B.Cu, net (none)
- added copper zone on F.Cu, net (none)
Other:
- board size 378.3 x 160.2 mm -> 183.8 x 130.2 mm
- board text removed: "FAT-O-TESA SPLIT KEYBOARD v0.1 - 2023"
- board text removed: "FAT-O-TESA SPLIT KEYBOARD v0.1 - 2023/24"
- board text removed: "created by stefangluszek"
