File: pcbs/v0.2/right/right.kicad_pcb (KiCad board)
At the start: 2 copper layers, 3.4 x 3 mm, 98 parts, among them SW1 RESET, SW2 RotaryEncoder_Switch, U1 ProMicro, U2 TRRS

Commit message: Routed PCB traces.
Parts:
- added G***: LOGO, LOGO, F.Cu at (107.9, 38.9)
- D1, D10, D11, D12, D13, D14, D15, D16, D17, D18, D19, D2, D20, D21, D22, D23, D24, D25, D26, D27, D28, D29, D3, D30, D31, D32, D33, D34, D35, D36, D37, D4, D5, D6, D7, D8, D9, SW1: moved to B.Cu
- D38, D39, D40, D41, D42, D43: footprint Keebio-Parts:SK6812-MINI-E -> LED_SMD:LED_WS2812B_PLCC4_5.0x5.0mm_P3.2mm; moved to B.Cu
- moved H6 428.4 mm to (40.5, 96.0)
- moved D42 421.3 mm to (42.1, 35.7), turned to 180 degrees
- moved SW1 418.9 mm to (42.1, 65.1), turned to -90 degrees
- moved H8 404.0 mm to (36.5, 51.6)
- moved H10 394.9 mm to (36.5, 129.4)
- moved H5 391.8 mm to (64.3, 132.5)
- moved D43 383.8 mm to (57.1, 145.2), turned to 180 degrees
- moved H1 380.3 mm to (99.2, 49.2)
- moved U2 380.2 mm to (88.9, 29.5)
- moved U1 376.2 mm to (65.5, 42.1), turned to 90 degrees
- moved H7 361.0 mm to (119.1, 92.9)
- moved D40 331.8 mm to (134.9, 34.9), turned to 180 degrees
- moved H3 327.4 mm to (128.6, 131.8)
- moved D19 307.6 mm to (57.1, 87.1), turned to 90 degrees
- moved H2 306.1 mm to (175.4, 76.2)
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Connections:
- D38 pad 1: Net-(D38-DOUT) -> VCC
- D38 pad 2: GND -> Net-(D38-VSS)
- D38 pad 3: Net-(D38-DIN) -> GND
- D38 pad 4: VCC -> Net-(D38-VDD)
- D39 pad 1: Net-(D39-DOUT) -> VCC
- D39 pad 2: GND -> Net-(D39-VSS)
- D39 pad 3: Net-(D38-DOUT) -> GND
- D39 pad 4: VCC -> Net-(D38-VSS)
- D40 pad 1: Net-(D38-DIN) -> VCC
- D40 pad 2: GND -> Net-(D38-VDD)
- D40 pad 3: Net-(D40-DIN) -> GND
- D40 pad 4: VCC -> Net-(D40-VDD)
- D41 pad 1: Net-(D41-DOUT) -> VCC
- D41 pad 2: GND -> Net-(D41-VSS)
- D41 pad 3: Net-(D39-DOUT) -> GND
- D41 pad 4: VCC -> Net-(D39-VSS)
- D42 pad 1: Net-(D40-DIN) -> VCC
- D42 pad 2: GND -> Net-(D40-VDD)
- D42 pad 3: LED -> GND
- D42 pad 4: VCC -> LED
- D43 pad 1: unconnected-(D43-DOUT-Pad1) -> VCC
- D43 pad 2: GND -> unconnected-(D43-DOUT-Pad2)
- D43 pad 3: Net-(D41-DOUT) -> GND
- D43 pad 4: VCC -> Net-(D41-VSS)
- U1 pad 10: row2 -> row1
- U1 pad 11: row1 -> row4
- U1 pad 12: row0 -> row5
- U1 pad 20: col3 -> col4
- U1 pad 21: col4 -> col5
- U1 pad 22: col5 -> col6
- U1 pad 23: col6 -> col7
- U1 pad 24: col7 -> row0
- U1 pad 7: row5 -> row2
- U1 pad 8: row4 -> col3
Routing:
- net VCC: track 0.00 -> 413.8 mm
- net row4: track 0.00 -> 244.9 mm, vias 0 -> 13
- net row5: track 0.00 -> 240.0 mm, vias 0 -> 10
- net col7: track 0.00 -> 231.5 mm, vias 0 -> 8
- net col6: track 0.00 -> 228.7 mm, vias 0 -> 4
- net col5: track 0.00 -> 212.2 mm, vias 0 -> 4
- net row3: track 0.00 -> 198.0 mm, vias 0 -> 11
- net row2: track 0.00 -> 192.0 mm, vias 0 -> 16
- net col4: track 0.00 -> 188.9 mm
- net row1: track 0.00 -> 173.5 mm, vias 0 -> 12
- net encA: track 0.00 -> 136.4 mm, vias 0 -> 4
- net col2: track 0.00 -> 134.3 mm
- net Net-(D38-VSS): track 0.00 -> 133.7 mm, vias 0 -> 12
- net col3: track 0.00 -> 128.3 mm
- net encB: track 0.00 -> 127.6 mm, vias 0 -> 10
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- added copper zone on B.Cu, net (none)
- added copper zone on F.Cu, net GND
Other:
- board size 3.4 x 3 mm -> 178.7 x 122.2 mm
