File: pcbs/v0.2/left/v0.2.kicad_pcb (KiCad board)
At the start: 2 copper layers, 182.6 x 119.1 mm, 94 parts, among them J1 OLED_128x32, SW2 RESET, U1 ProMicro, U2 TRRS

Commit message: v0.2 - Left - Updated LEDs Symbols.
NOTE: This caused the traces to no longer match the footprint and thus
removed.

MISSING TRACES!
Parts:
- D37, D38, D39, D40, D41, D42: footprint Keebio-Parts:WS2812B -> LED_SMD:LED_SK6812MINI_PLCC4_3.5x3.5mm_P1.75mm
Routing:
- net VCC: track 350.7 -> 0.00 mm, vias 10 -> 0
- net col2: track 221.4 -> 0.00 mm, vias 4 -> 0
- net col4: track 209.4 -> 0.00 mm, vias 6 -> 0
- net row4: track 209.2 -> 0.00 mm, vias 10 -> 0
- net row5: track 208.9 -> 0.00 mm
- net col5: track 194.9 -> 0.00 mm, vias 8 -> 0
- net col6: track 194.7 -> 0.00 mm, vias 12 -> 0
- net col3: track 181.7 -> 0.00 mm, vias 4 -> 0
- net row3: track 180.9 -> 0.00 mm, vias 11 -> 0
- net /TRRS-data: track 160.4 -> 0.00 mm, vias 2 -> 0
- net row1: track 159.1 -> 0.00 mm, vias 14 -> 0
- net row2: track 156.8 -> 0.00 mm, vias 12 -> 0
- net col1: track 135.6 -> 0.00 mm, vias 2 -> 0
- net row0: track 133.4 -> 0.00 mm, vias 10 -> 0
- net col0: track 114.6 -> 0.00 mm
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- removed copper zone on B.Cu, net (none)
- removed copper zone on F.Cu, net GND
