File: pcbs/v0.2/left/v0.2.kicad_sch (KiCad schematic)
At the start: 81 parts, among them J2 TRRS, SW1 RotaryEncoder_Switch, SW2 RESET, U1 ProMicro

Commit message: v0.2 - Left - PCB.
Parts:
- removed D37, D38, D39, D40, D41, D42, D43, D44, D45, D46, D47, D48, D49, D50, D51, D52, D53, D54, D55, D56, D57, D58, D59, D60, D61, D62, D63, D64, D65, D66, D67, D68, D69, D70, D71, D72: Diode, Keebio-Parts:Diode, symbol ScottoKeebs:Placeholder_Diode
- removed J2: TRRS, Keebio-Parts:RotaryEncoder_EC11, symbol Connector_Audio:AudioJack4
- removed MX1, MX38, MX39, MX40, MX41, MX42, MX44, MX45, MX46, MX47, MX48, MX49, MX50, MX51, MX52, MX53, MX54, MX55, MX56, MX57, MX58, MX59, MX60, MX61, MX62, MX63, MX64, MX65, MX66, MX67, MX68, MX69, MX70, MX71, MX72: MX_SW_solder, marbastlib-mx:SW_MX_1u, symbol marbastlib-mx:MX_SW_solder
- removed SW1: RotaryEncoder_Switch, Keebio-Parts:RotaryEncoder_EC11, symbol Device:RotaryEncoder_Switch
- added D1, D10, D11, D12, D13, D14, D15, D16, D17, D18, D19, D2, D20, D21, D22, D23, D24, D25, D26, D27, D28, D29, D3, D30, D31, D32, D33, D34, D35, D36, D4, D5, D6, D7, D8, D9: Diode, Diode_THT:D_DO-35_SOD27_P7.62mm_Horizontal, symbol ScottoKeebs:Placeholder_Diode
- added H1, H11, H12, H13, H14, H15, H6: MountingHole, MountingHole:MountingHole_4.3mm_M4, symbol Mechanical:MountingHole
- added H10, H7, H8, H9: MountingHole, MountingHole:MountingHole_5.3mm_M5, symbol Mechanical:MountingHole
- added J1: OLED_128x32, ScottoKeebs_Components:OLED_128x32, symbol ScottoKeebs:OLED_128x32
- added MX1, MX10, MX11, MX12, MX14, MX15, MX16, MX17, MX18, MX2, MX20, MX21, MX22, MX23, MX24, MX26, MX27, MX28, MX29, MX3, MX30, MX31, MX36, MX4, MX5, MX6, MX7, MX8, MX9: MX_SW_HS, ScottoKeebs_MX:MX_PCB_1.00u, symbol marbastlib-mx:MX_SW_HS
- added MX13: MX_SW_HS, ScottoKeebs_MX:MX_PCB_1.50u, symbol marbastlib-mx:MX_SW_HS
- added MX19, MX35: MX_SW_HS, ScottoKeebs_MX:MX_PCB_1.75u, symbol marbastlib-mx:MX_SW_HS
- added MX25, MX32, MX33, MX34: MX_SW_HS, ScottoKeebs_MX:MX_PCB_1.25u, symbol marbastlib-mx:MX_SW_HS
- added U2: TRRS, ScottoKeebs_Components:TRRS_PJ-320A, symbol ScottoKeebs:Placeholder_TRRS
- D37: renamed from D1; footprint LED_SMD:LED_SK6812MINI_PLCC4_3.5x3.5mm_P1.75mm -> Keebio-Parts:WS2812B
- D38: renamed from D2; footprint LED_SMD:LED_SK6812MINI_PLCC4_3.5x3.5mm_P1.75mm -> Keebio-Parts:WS2812B
- D39: renamed from D3; footprint LED_SMD:LED_SK6812MINI_PLCC4_3.5x3.5mm_P1.75mm -> Keebio-Parts:WS2812B
- D40: renamed from D4; footprint LED_SMD:LED_SK6812MINI_PLCC4_3.5x3.5mm_P1.75mm -> Keebio-Parts:WS2812B
- D41: renamed from D5; footprint LED_SMD:LED_SK6812MINI_PLCC4_3.5x3.5mm_P1.75mm -> Keebio-Parts:WS2812B
- D42: renamed from D6; footprint LED_SMD:LED_SK6812MINI_PLCC4_3.5x3.5mm_P1.75mm -> Keebio-Parts:WS2812B
- U1: footprint PCM_marbastlib-xp-promicroish:ProMicro_USBup -> marbastlib-xp-promicroish:ProMicro_Reversible_Single
Connections:
- net GND: now also J1.1 (GND), U2.1 (SLEEVE)
- net VCC: now also J1.2 (VCC), U2.3 (RING1)
- net col0: now also MX1.1, MX13.1, MX19.1, MX25.1, MX32.1, MX6.1
- net col1: now also MX14.1, MX20.1, MX26.1, MX33.1, MX7.1
- net col2: now also MX15.1, MX2.1, MX21.1, MX27.1, MX34.1, MX8.1
- net col3: now also MX16.1, MX22.1, MX28.1, MX3.1, MX35.1, MX9.1
- net col4: now also MX10.1, MX17.1, MX23.1, MX29.1, MX36.1, MX4.1
- net col5: now also MX11.1, MX18.1, MX24.1, MX30.1, MX5.1
- net col6: now also MX12.1, MX31.1
- net row0: now also D1.1 (K), D2.1 (K), D3.1 (K), D4.1 (K), D5.1 (K)
- net row1: now also D10.1 (K), D11.1 (K), D12.1 (K), D6.1 (K), D7.1 (K), D8.1 (K), D9.1 (K)
- net row2: now also D13.1 (K), D14.1 (K), D15.1 (K), D16.1 (K), D17.1 (K), D18.1 (K)
- net row3: now also D19.1 (K), D20.1 (K), D21.1 (K), D22.1 (K), D23.1 (K), D24.1 (K)
- net row4: now also D25.1 (K), D26.1 (K), D27.1 (K), D28.1 (K), D29.1 (K), D30.1 (K), D31.1 (K)
- net row5: now also D32.1 (K), D33.1 (K), D34.1 (K), D35.1 (K), D36.1 (K)
- net RST: now reaches SW2.1, U1.15 (RST)
- net TRRS-data: now reaches U1.2 (D2-RX)
- net TRRS-data: now also U2.4 (RING2)
- net encA renamed SDA
- net SDA: now also J1.4 (SDA)
- net encB renamed SCL
- net SCL: now also J1.3 (SCL)
- new net: D28.2 (A), MX28.2
- new net: D13.2 (A), MX13.2
- new net: D3.2 (A), MX3.2
- new net: D12.2 (A), MX12.2
- new net: D18.2 (A), MX18.2
- new net: D21.2 (A), MX21.2
- new net: D17.2 (A), MX17.2
- new net: D26.2 (A), MX26.2
- new net: D22.2 (A), MX22.2
- new net: D35.2 (A), MX35.2
- new net: D33.2 (A), MX33.2
- new net: D1.2 (A), MX1.2
- new net: D32.2 (A), MX32.2
- new net: D29.2 (A), MX29.2
- new net: D25.2 (A), MX25.2
- new net: D8.2 (A), MX8.2
- new net: D36.2 (A), MX36.2
- new net: D27.2 (A), MX27.2
- new net: D34.2 (A), MX34.2
- new net: D5.2 (A), MX5.2
- new net: D14.2 (A), MX14.2
- new net: D6.2 (A), MX6.2
- new net: D2.2 (A), MX2.2
- new net: D23.2 (A), MX23.2
- new net: D10.2 (A), MX10.2
- new net: D9.2 (A), MX9.2
- new net: D4.2 (A), MX4.2
- new net: D19.2 (A), MX19.2
- new net: D11.2 (A), MX11.2
- new net: D31.2 (A), MX31.2
- new net: D15.2 (A), MX15.2
- new net: D24.2 (A), MX24.2
- new net: D20.2 (A), MX20.2
- new net: D16.2 (A), MX16.2
- new net: D7.2 (A), MX7.2
- new net: D30.2 (A), MX30.2
Other:
- note added: "Keyboard matrix [6x7]"
- note added: "Underglow LEDs"
- note added: "plate mounts"
- note added: "tenting"

Commit message: v0.2 - Left - Updated LEDs Symbols.
NOTE: This caused the traces to no longer match the footprint and thus
removed.

MISSING TRACES!
Parts:
- D37, D38, D39, D40, D41, D42: footprint Keebio-Parts:WS2812B -> LED_SMD:LED_SK6812MINI_PLCC4_3.5x3.5mm_P1.75mm
Changed lines of the file:
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@@
       (effects (font (size 1.27 1.27)) hide)
     )
-    (property "Footprint" "Keebio-Parts:WS2812B" (at 224.79 111.76 0)
+    (property "Footprint" "LED_SMD:LED_SK6812MINI_PLCC4_3.5x3.5mm_P1.75mm" (at 224.79 111.76 0)
       (effects (font (size 1.27 1.27)) (justify left top) hide)
     )
@@
       (effects (font (size 1.27 1.27)) hide)
     )
-    (property "Footprint" "Keebio-Parts:WS2812B" (at 179.07 111.76 0)
+    (property "Footprint" "LED_SMD:LED_SK6812MINI_PLCC4_3.5x3.5mm_P1.75mm" (at 179.07 111.76 0)
       (effects (font (size 1.27 1.27)) (justify left top) hide)
     )
@@
       (effects (font (size 1.27 1.27)) hide)
     )
-    (property "Footprint" "Keebio-Parts:WS2812B" (at 181.61 148.59 0)
+    (property "Footprint" "LED_SMD:LED_SK6812MINI_PLCC4_3.5x3.5mm_P1.75mm" (at 181.61 148.59 0)
       (effects (font (size 1.27 1.27)) (justify left top) hide)
     )
@@
       (effects (font (size 1.27 1.27)) hide)
     )
-    (property "Footprint" "Keebio-Parts:WS2812B" (at 227.33 148.59 0)
+    (property "Footprint" "LED_SMD:LED_SK6812MINI_PLCC4_3.5x3.5mm_P1.75mm" (at 227.33 148.59 0)
       (effects (font (size 1.27 1.27)) (justify left top) hide)
     )
@@
       (effects (font (size 1.27 1.27)) hide)
     )
-    (property "Footprint" "Keebio-Parts:WS2812B" (at 205.74 148.59 0)
+    (property "Footprint" "LED_SMD:LED_SK6812MINI_PLCC4_3.5x3.5mm_P1.75mm" (at 205.74 148.59 0)
       (effects (font (size 1.27 1.27)) (justify left top) hide)
     )
@@
       (effects (font (size 1.27 1.27)) hide)
     )
-    (property "Footprint" "Keebio-Parts:WS2812B" (at 203.2 111.76 0)
+    (property "Footprint" "LED_SMD:LED_SK6812MINI_PLCC4_3.5x3.5mm_P1.75mm" (at 203.2 111.76 0)
       (effects (font (size 1.27 1.27)) (justify left top) hide)
     )
